File: pcb/wasdpad.kicad_sch (KiCad schematic)
At the start: 24 parts, among them SW1 SW_Push_45deg, SW2 SW_Push_45deg, SW3 SW_Push_45deg, SW4 SW_Push_45deg, SW5 SW_Push_45deg, SW6 SW_Push_45deg, U1 XIAO-RP2040-DIP

Commit message: fix unconnected neopixel
Connections:
- net at D13.3 (DIN): now also D6.1 (DOUT)
Changed lines of the file:
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@@
+	(wire
+		(pts
+			(xy 69.85 163.83) (xy 119.38 163.83)
+		)
+		(stroke
+			(width 0)
+			(type default)
+		)
+	)
 	(wire
 		(pts

Commit message: add production files
Other:
- note added: "Neopixels"
- note added: "OLED"
- note added: "Switch Matrix"
- note added: "XIAO"
- moved on the sheet: Brd1, D1, D10, D11, D12, D13, D14, D2, D3, D4, D5, D6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
